File: 4H-RGBLight.brd (EAGLE design)
At the start: 30.5 x 35.6 mm, 9 parts

Commit message: from Makefile
Parts:
- U$3: value 4H-LOGO6 -> (none)
Changed lines of the file:
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@@
 <element name="S3" library="barbary_enterprises" package="TACTILE-PTH" value="" x="24.765" y="21.59" smashed="yes" rot="R180"/>
 <element name="LED3" library="barbary_enterprises" package="LED-OVAL" value="BLUE" x="20.32" y="31.75"/>
-<element name="U$3" library="4h" package="4H_LOGO_6" value="4H-LOGO6" x="15.24" y="8.763" rot="MR0"/>
+<element name="U$3" library="4h" package="4H_LOGO_6" value="" x="15.24" y="8.763" rot="MR0"/>
 </elements>
 <signals>
