File: RGB_Light.brd (EAGLE design)
At the start: 30.5 x 35.6 mm, 9 parts

Commit message: from Makefile
Parts:
- R1: value 50 -> 51
Changed lines of the file:
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@@
 <attribute name="VALUE" x="19.558" y="13.97" size="1.6764" layer="27" font="vector" rot="R180"/>
 </element>
-<element name="R1" library="barbary_enterprises" package="AXIAL-0.3" value="50" x="6.35" y="26.67" rot="R180"/>
+<element name="R1" library="barbary_enterprises" package="AXIAL-0.3" value="51" x="6.35" y="26.67" rot="R180"/>
 <element name="S2" library="barbary_enterprises" package="TACTILE-PTH" value="" x="15.24" y="21.59" smashed="yes" rot="R180"/>
 <element name="LED2" library="barbary_enterprises" package="LED-OVAL" value="GREEN" x="15.24" y="31.75"/>

Commit message: from Makefile
Parts:
- LED1, LED2, LED3: device barbary_enterprises:LED-OVAL -> barbary_enterprises:LED5MM
- moved LED1 1.28 mm to (8.89, 31.6), turned to 180 degrees
- moved LED3 1.27 mm to (21.6, 31.8), turned to 180 degrees
- turned LED2 to 180 degrees
- renumbered U$2 to B1
Connections:
- net GND: now also LED1.K, LED2.K, LED3.K; no longer LED1.CATHODE, LED2.CATHODE, LED3.CATHODE
- net N$1: now also LED2.A; no longer LED2.ANODE
- net N$3: now also LED3.A; no longer LED3.ANODE
- net N$4: now also LED1.A; no longer LED1.ANODE
Routing:
- net GND: track 38.4 -> 39.4 mm
- net N$4: track 5.61 -> 4.95 mm
- net N$3: track 14.4 -> 15.0 mm
Changed lines of the file:
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@@
 </autorouter>
 <elements>
-<element name="LED1" library="barbary_enterprises" package="LED-OVAL" value="RED" x="10.16" y="31.75"/>
+<element name="LED1" library="barbary_enterprises" package="LED5MM" value="RED" x="8.89" y="31.623" smashed="yes" rot="R180">
+<attribute name="NAME" x="8.89" y="29.083" size="1.27" layer="26" ratio="10" rot="MR180" align="top-center"/>
+<attribute name="VALUE" x="8.89" y="33.02" size="1.27" layer="28" ratio="10" rot="MR180" align="top-center"/>
+</element>
 <element name="S1" library="barbary_enterprises" package="TACTILE-PTH" value="" x="5.842" y="21.59" smashed="yes" rot="R180"/>
-<element name="U$2" library="battery" package="CR2032-THRU" value="" x="15.24" y="7.62" smashed="yes" rot="R180">
+<element name="B1" library="battery" package="CR2032-THRU" value="" x="15.24" y="7.62" smashed="yes" rot="R180">
 <attribute name="VALUE" x="19.558" y="13.97" size="1.6764" layer="27" font="vector" rot="R180"/>
 </element>
 <element name="R1" library="barbary_enterprises" package="AXIAL-0.3" value="51" x="6.35" y="26.67" rot="R180"/>
 <element name="S2" library="barbary_enterprises" package="TACTILE-PTH" value="" x="15.24" y="21.59" smashed="yes" rot="R180"/>
-<element name="LED2" library="barbary_enterprises" package="LED-OVAL" value="GREEN" x="15.24" y="31.75"/>
+<element name="LED2" library="barbary_enterprises" package="LED5MM" value="GREEN" x="15.24" y="31.75" smashed="yes" rot="R180">
+<attribute name="NAME" x="15.24" y="29.083" size="1.27" layer="26" ratio="10" rot="MR180" align="top-center"/>
+<attribute name="VALUE" x="15.24" y="33.02" size="1.27" layer="28" ratio="10" rot="MR180" align="top-center"/>
+</element>
 <element name="S3" library="barbary_enterprises" package="TACTILE-PTH" value="" x="24.765" y="21.59" smashed="yes" rot="R180"/>
-<element name="LED3" library="barbary_enterprises" package="LED-OVAL" value="BLUE" x="20.32" y="31.75"/>
+<element name="LED3" library="barbary_enterprises" package="LED5MM" value="BLUE" x="21.59" y="31.75" smashed="yes" rot="R180">
+<attribute name="NAME" x="21.59" y="28.956" size="1.27" layer="26" ratio="10" rot="MR180" align="top-center"/>
+<attribute name="VALUE" x="21.59" y="33.02" size="1.27" layer="28" ratio="10" rot="MR180" align="top-center"/>
+</element>
 <element name="U$1" library="logo" package="USER_HACKABLE" value="USER_HACKABLE" x="15.24" y="8.763" rot="MR0"/>
 </elements>
 <signals>
 <signal name="GND">
-<contactref element="LED1" pad="CATHODE"/>
-<contactref element="U$2" pad="-"/>
-<contactref element="LED2" pad="CATHODE"/>
-<contactref element="LED3" pad="CATHODE"/>
+<contactref element="LED1" pad="K"/>
+<contactref element="B1" pad="-"/>
+<contactref element="LED2" pad="K"/>
+<contactref element="LED3" pad="K"/>
 <wire x1="15.24" y1="7.62" x2="15.24" y2="29.21" width="0.8128" layer="1"/>
 <wire x1="15.24" y1="29.21" x2="13.97" y2="30.48" width="0.8128" layer="1"/>
 <wire x1="13.97" y1="30.48" x2="13.97" y2="31.75" width="0.8128" layer="1"/>
-<wire x1="8.89" y1="31.75" x2="8.89" y2="30.48" width="0.8128" layer="1"/>
+<wire x1="7.62" y1="31.623" x2="8.89" y2="30.48" width="0.8128" layer="1"/>
 <wire x1="8.89" y1="30.48" x2="10.16" y2="29.21" width="0.8128" layer="1"/>
 <wire x1="10.16" y1="29.21" x2="15.24" y2="29.21" width="0.8128" layer="1"/>
-<wire x1="19.05" y1="31.75" x2="19.05" y2="30.48" width="0.8128" layer="1"/>
-<wire x1="19.05" y1="30.48" x2="17.78" y2="29.21" width="0.8128" layer="1"/>
+<wire x1="20.32" y1="31.75" x2="17.78" y2="29.21" width="0.8128" layer="1"/>
 <wire x1="17.78" y1="29.21" x2="15.24" y2="29.21" width="0.8128" layer="1"/>
 </signal>
 <signal name="V_BATT">
 <contactref element="S1" pad="1"/>
-<contactref element="U$2" pad="+2"/>
-<contactref element="U$2" pad="+1"/>
+<contactref element="B1" pad="+2"/>
+<contactref element="B1" pad="+1"/>
 <contactref element="S3" pad="1"/>
 <contactref element="S2" pad="1"/>
@@
 <signal name="N$1">
 <contactref element="S2" pad="3"/>
-<contactref element="LED2" pad="ANODE"/>
+<contactref element="LED2" pad="A"/>
 <contactref element="S2" pad="4"/>
 <wire x1="11.9888" y1="23.8506" x2="16.51" y2="23.8506" width="0.8128" layer="16"/>
@@
 <signal name="N$3">
 <contactref element="S3" pad="3"/>
-<contactref element="LED3" pad="ANODE"/>
+<contactref element="LED3" pad="A"/>
 <contactref element="S3" pad="4"/>
 <wire x1="28.0162" y1="23.8506" x2="21.5138" y2="23.8506" width="0.8128" layer="16"/>
-<wire x1="21.59" y1="31.75" x2="21.59" y2="23.9268" width="0.8128" layer="16"/>
+<wire x1="22.86" y1="31.75" x2="22.86" y2="29.21" width="0.8128" layer="16"/>
+<wire x1="22.86" y1="29.21" x2="21.59" y2="27.94" width="0.8128" layer="16"/>
+<wire x1="21.59" y1="27.94" x2="21.59" y2="23.9268" width="0.8128" layer="16"/>
 <wire x1="21.59" y1="23.9268" x2="21.5138" y2="23.8506" width="0.8128" layer="16"/>
 </signal>
 <signal name="N$4">
-<contactref element="LED1" pad="ANODE"/>
+<contactref element="LED1" pad="A"/>
 <contactref element="R1" pad="P$1"/>
-<wire x1="11.43" y1="31.75" x2="11.43" y2="27.94" width="0.8128" layer="16"/>
-<wire x1="11.43" y1="27.94" x2="10.16" y2="26.67" width="0.8128" layer="16"/>
+<wire x1="10.16" y1="31.623" x2="10.16" y2="26.67" width="0.8128" layer="16"/>
 </signal>
 </signals>
