File: RGB_Light.sch (EAGLE design)
At the start: 9 parts

Commit message: from Makefile
Parts:
- removed U$3: (no value), 4h:4H-LOGO6
- added U$1: USER_HACKABLE, logo:USER_HACKABLE
Changed lines of the file:
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@@
 <part name="S3" library="barbary_enterprises" deviceset="TAC_SWITCH" device="PTH"/>
 <part name="LED3" library="barbary_enterprises" deviceset="LED" device="OVAL" value="BLUE"/>
-<part name="U$3" library="4h" deviceset="4H-LOGO" device="6"/>
+<part name="U$1" library="logo" deviceset="USER_HACKABLE" device=""/>
 </parts>
 <sheets>
@@
 <instance part="S3" gate="S" x="60.96" y="43.18" rot="R270"/>
 <instance part="LED3" gate="G$1" x="58.42" y="17.78"/>
-<instance part="U$3" gate="G$1" x="27.94" y="5.08"/>
+<instance part="U$1" gate="G$1" x="78.74" y="15.24"/>
 </instances>
 <busses>

Commit message: from Makefile
Parts:
- R1: value 50 -> 51
Changed lines of the file:
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@@
 <part name="LED1" library="barbary_enterprises" deviceset="LED" device="OVAL" value="RED"/>
 <part name="U$2" library="battery" deviceset="CR2032" device="THM"/>
-<part name="R1" library="barbary_enterprises" deviceset="RESISTOR" device="AXIAL-0.3" value="50"/>
+<part name="R1" library="barbary_enterprises" deviceset="RESISTOR" device="AXIAL-0.3" value="51"/>
 <part name="S2" library="barbary_enterprises" deviceset="TAC_SWITCH" device="PTH"/>
 <part name="LED2" library="barbary_enterprises" deviceset="LED" device="OVAL" value="GREEN"/>

Commit message: from Makefile
Parts:
- LED1, LED2, LED3: device barbary_enterprises:LEDOVAL -> barbary_enterprises:LED5MM
- renumbered U$2 to B1
Changed lines of the file:
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@@
 <grid distance="0.1" unitdist="inch" unit="inch" style="lines" multiple="1" display="no" altdistance="0.01" altunitdist="inch" altunit="inch"/>
 <layers>
-<layer number="1" name="Top" color="4" fill="1" visible="no" active="no"/>
-<layer number="16" name="Bottom" color="1" fill="1" visible="no" active="no"/>
-<layer number="17" name="Pads" color="2" fill="1" visible="no" active="no"/>
-<layer number="18" name="Vias" color="2" fill="1" visible="no" active="no"/>
-<layer number="19" name="Unrouted" color="6" fill="1" visible="no" active="no"/>
-<layer number="20" name="Dimension" color="15" fill="1" visible="no" active="no"/>
-<layer number="21" name="tPlace" color="7" fill="1" visible="no" active="no"/>
-<layer number="22" name="bPlace" color="7" fill="1" visible="no" active="no"/>
-<layer number="23" name="tOrigins" color="15" fill="1" visible="no" active="no"/>
-<layer number="24" name="bOrigins" color="15" fill="1" visible="no" active="no"/>
-<layer number="25" name="tNames" color="7" fill="1" visible="no" active="no"/>
-<layer number="26" name="bNames" color="7" fill="1" visible="no" active="no"/>
-<layer number="27" name="tValues" color="7" fill="1" visible="no" active="no"/>
-<layer number="28" name="bValues" color="7" fill="1" visible="no" active="no"/>
+<layer number="1" name="Top" color="4" fill="1" visible="yes" active="no"/>
+<layer number="16" name="Bottom" color="1" fill="1" visible="yes" active="no"/>
+<layer number="17" name="Pads" color="2" fill="1" visible="yes" active="no"/>
+<layer number="18" name="Vias" color="2" fill="1" visible="yes" active="no"/>
+<layer number="19" name="Unrouted" color="6" fill="1" visible="yes" active="no"/>
+<layer number="20" name="Dimension" color="15" fill="1" visible="yes" active="no"/>
+<layer number="21" name="tPlace" color="7" fill="1" visible="yes" active="no"/>
+<layer number="22" name="bPlace" color="14" fill="1" visible="yes" active="no"/>
+<layer number="23" name="tOrigins" color="15" fill="1" visible="yes" active="no"/>
+<layer number="24" name="bOrigins" color="14" fill="1" visible="yes" active="no"/>
+<layer number="25" name="tNames" color="7" fill="1" visible="yes" active="no"/>
+<layer number="26" name="bNames" color="14" fill="1" visible="yes" active="no"/>
+<layer number="27" name="tValues" color="7" fill="1" visible="yes" active="no"/>
+<layer number="28" name="bValues" color="14" fill="1" visible="yes" active="no"/>
 <layer number="29" name="tStop" color="7" fill="3" visible="no" active="no"/>
 <layer number="30" name="bStop" color="7" fill="6" visible="no" active="no"/>
@@
 <layer number="35" name="tGlue" color="7" fill="4" visible="no" active="no"/>
 <layer number="36" name="bGlue" color="7" fill="5" visible="no" active="no"/>
-<layer number="37" name="tTest" color="7" fill="1" visible="no" active="no"/>
-<layer number="38" name="bTest" color="7" fill="1" visible="no" active="no"/>
+<layer number="37" name="tTest" color="7" fill="1" visible="yes" active="no"/>
+<layer number="38" name="bTest" color="7" fill="1" visible="yes" active="no"/>
 <layer number="39" name="tKeepout" color="4" fill="11" visible="no" active="no"/>
 <layer number="40" name="bKeepout" color="1" fill="11" visible="no" active="no"/>
@@
 <layer number="44" name="Drills" color="7" fill="1" visible="no" active="no"/>
 <layer number="45" name="Holes" color="7" fill="1" visible="no" active="no"/>
-<layer number="46" name="Milling" color="3" fill="1" visible="no" active="no"/>
-<layer number="47" name="Measures" color="7" fill="1" visible="no" active="no"/>
-<layer number="48" name="Document" color="7" fill="1" visible="no" active="no"/>
-<layer number="49" name="Reference" color="7" fill="1" visible="no" active="no"/>
-<layer number="50" name="dxf" color="7" fill="1" visible="no" active="no"/>
-<layer number="51" name="tDocu" color="7" fill="1" visible="no" active="no"/>
-<layer number="52" name="bDocu" color="7" fill="1" visible="no" active="no"/>
-<layer number="53" name="tGND_GNDA" color="7" fill="9" visible="no" active="no"/>
-<layer number="54" name="bGND_GNDA" color="1" fill="9" visible="no" active="no"/>
-<layer number="56" name="wert" color="7" fill="1" visible="no" active="no"/>
-<layer number="57" name="tCAD" color="7" fill="1" visible="no" active="no"/>
-<layer number="59" name="tCarbon" color="7" fill="1" visible="no" active="no"/>
-<layer number="60" name="bCarbon" color="7" fill="1" visible="no" active="no"/>
+<layer number="46" name="Milling" color="3" fill="1" visible="yes" active="no"/>
+<layer number="47" name="Measures" color="7" fill="1" visible="yes" active="no"/>
+<layer number="48" name="Document" color="7" fill="1" visible="yes" active="no"/>
+<layer number="49" name="Reference" color="7" fill="1" visible="yes" active="no"/>
+<layer number="50" name="dxf" color="7" fill="1" visible="yes" active="no"/>
+<layer number="51" name="tDocu" color="7" fill="1" visible="yes" active="no"/>
+<layer number="52" name="bDocu" color="14" fill="1" visible="yes" active="no"/>
+<layer number="53" name="tGND_GNDA" color="7" fill="9" visible="yes" active="no"/>
+<layer number="54" name="bGND_GNDA" color="1" fill="9" visible="yes" active="no"/>
+<layer number="56" name="wert" color="7" fill="1" visible="yes" active="no"/>
+<layer number="57" name="tCAD" color="7" fill="1" visible="yes" active="no"/>
+<layer number="59" name="tCarbon" color="7" fill="1" visible="yes" active="no"/>
+<layer number="60" name="bCarbon" color="7" fill="1" visible="yes" active="no"/>
 <layer number="90" name="Modules" color="5" fill="1" visible="yes" active="yes"/>
 <layer number="91" name="Nets" color="2" fill="1" visible="yes" active="yes"/>
@@
 <part name="SUPPLY1" library="SparkFun-Aesthetics" deviceset="V_BATT" device=""/>
 <part name="S1" library="barbary_enterprises" deviceset="TAC_SWITCH" device="PTH"/>
-<part name="LED1" library="barbary_enterprises" deviceset="LED" device="OVAL" value="RED"/>
-<part name="U$2" library="battery" deviceset="CR2032" device="THM"/>
+<part name="LED1" library="barbary_enterprises" deviceset="LED" device="5MM" value="RED"/>
+<part name="B1" library="battery" deviceset="CR2032" device="THM"/>
 <part name="R1" library="barbary_enterprises" deviceset="RESISTOR" device="AXIAL-0.3" value="51"/>
 <part name="S2" library="barbary_enterprises" deviceset="TAC_SWITCH" device="PTH"/>
-<part name="LED2" library="barbary_enterprises" deviceset="LED" device="OVAL" value="GREEN"/>
+<part name="LED2" library="barbary_enterprises" deviceset="LED" device="5MM" value="GREEN"/>
 <part name="S3" library="barbary_enterprises" deviceset="TAC_SWITCH" device="PTH"/>
-<part name="LED3" library="barbary_enterprises" deviceset="LED" device="OVAL" value="BLUE"/>
+<part name="LED3" library="barbary_enterprises" deviceset="LED" device="5MM" value="BLUE"/>
 <part name="U$1" library="logo" deviceset="USER_HACKABLE" device=""/>
 </parts>
@@
 <instance part="S1" gate="S" x="25.4" y="43.18" rot="R270"/>
 <instance part="LED1" gate="G$1" x="22.86" y="17.78"/>
-<instance part="U$2" gate="G$1" x="15.24" y="43.18" rot="R90"/>
+<instance part="B1" gate="G$1" x="15.24" y="43.18" rot="R90"/>
 <instance part="R1" gate="G$1" x="22.86" y="27.94" rot="R90"/>
 <instance part="S2" gate="S" x="43.18" y="43.18" rot="R270"/>
@@
 <wire x1="22.86" y1="12.7" x2="22.86" y2="10.16" width="0.1524" layer="91"/>
 <wire x1="22.86" y1="10.16" x2="15.24" y2="10.16" width="0.1524" layer="91"/>
-<pinref part="U$2" gate="G$1" pin="-"/>
+<pinref part="B1" gate="G$1" pin="-"/>
 <wire x1="15.24" y1="10.16" x2="10.16" y2="10.16" width="0.1524" layer="91"/>
 <wire x1="15.24" y1="38.1" x2="15.24" y2="10.16" width="0.1524" layer="91"/>
@@
 <wire x1="17.78" y1="50.8" x2="12.7" y2="50.8" width="0.1524" layer="91"/>
 <wire x1="12.7" y1="50.8" x2="10.16" y2="50.8" width="0.1524" layer="91"/>
-<pinref part="U$2" gate="G$1" pin="+1"/>
+<pinref part="B1" gate="G$1" pin="+1"/>
 <wire x1="17.78" y1="48.26" x2="17.78" y2="50.8" width="0.1524" layer="91"/>
 <junction x="17.78" y="50.8"/>
-<pinref part="U$2" gate="G$1" pin="+"/>
+<pinref part="B1" gate="G$1" pin="+"/>
 <wire x1="12.7" y1="48.26" x2="12.7" y2="50.8" width="0.1524" layer="91"/>
 <junction x="12.7" y="50.8"/>
